Commit message: updated files for vm

File: ur5e_urdf/urdf/ur5e_complete.urdf (robot description, URDF)
Before this commit: robot ur5e_mics_complete, 21 links, 20 joints
Links:
- link base_link_inertia: geometry collision mesh filename=/home/barutta/Robotic_liquid_pouring/ur5e_urdf/meshes/ur5e/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; visual mesh filename=/home/barutta/Robotic_liquid_pouring/ur5e_urdf/meshes/ur5e/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
- link forearm_link: geometry collision mesh filename=/home/barutta/Robotic_liquid_pouring/ur5e_urdf/meshes/ur5e/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; visual mesh filename=/home/barutta/Robotic_liquid_pouring/ur5e_urdf/meshes/ur5e/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
- link hand_e_link: geometry collision mesh filename=/home/barutta/Robotic_liquid_pouring/ur5e_urdf/meshes/robot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 scale=1.0 1.0 1.0; visual mesh filename=/home/barutta/Robotic_liquid_pouring/ur5e_urdf/meshes/robot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 scale=1.0 1.0 1.0
- link hande_left_finger: geometry collision mesh filename=/home/barutta/Robotic_liquid_pouring/ur5e_urdf/meshes/robot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 scale=1.0 1.0 1.0; visual mesh filename=/home/barutta/Robotic_liquid_pouring/ur5e_urdf/meshes/robot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 scale=1.0 1.0 1.0
- link hande_right_finger: geometry collision mesh filename=/home/barutta/Robotic_liquid_pouring/ur5e_urdf/meshes/robot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 scale=1.0 1.0 1.0; visual mesh filename=/home/barutta/Robotic_liquid_pouring/ur5e_urdf/meshes/robot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 scale=1.0 1.0 1.0
- link shoulder_link: geometry collision mesh filename=/home/barutta/Robotic_liquid_pouring/ur5e_urdf/meshes/ur5e/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; visual mesh filename=/home/barutta/Robotic_liquid_pouring/ur5e_urdf/meshes/ur5e/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
- link tabletop: geometry collision box size=1.18 0.95 0.9165; visual mesh filename=/home/barutta/Robotic_liquid_pouring/ur5e_urdf/meshes/extra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 scale=0.001 0.001 0.001
- link upper_arm_link: geometry collision mesh filename=/home/barutta/Robotic_liquid_pouring/ur5e_urdf/meshes/ur5e/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; visual mesh filename=/home/barutta/Robotic_liquid_pouring/ur5e_urdf/meshes/ur5e/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
- link wrist_1_link: geometry collision mesh filename=/home/barutta/Robotic_liquid_pouring/ur5e_urdf/meshes/ur5e/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; visual mesh filename=/home/barutta/Robotic_liquid_pouring/ur5e_urdf/meshes/ur5e/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
- link wrist_2_link: geometry collision mesh filename=/home/barutta/Robotic_liquid_pouring/ur5e_urdf/meshes/ur5e/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; visual mesh filename=/home/barutta/Robotic_liquid_pouring/ur5e_urdf/meshes/ur5e/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
- link wrist_3_link: geometry collision mesh filename=/home/barutta/Robotic_liquid_pouring/ur5e_urdf/meshes/ur5e/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; visual mesh filename=/home/barutta/Robotic_liquid_pouring/ur5e_urdf/meshes/ur5e/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
